Commit message: Configuration changed for jazzy

File: urdf/ikea_table.urdf (robot description, URDF)
Before this commit: robot ikea_table, 10 links, 9 joints
Links:
- removed link lidar
- added link chassis, mass 4.00000000; collision mesh filename=file:///home/andi/project/ros2_workspace/install/self_drivi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 scale=1 1 1; visual mesh filename=file:///home/andi/project/ros2_workspace/install/self_drivi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 scale=1 1 1
- added link control, mass 1.0; collision box size=0.075 0.25 0.075; visual box size=0.075 0.25 0.075
- added link rplidar_link, mass 0.1; collision cylinder length=0.02 radius=0.065; visual cylinder length=0.02 radius=0.065
- link base_footprint: mass None -> 0.0001; geometry visual box size=0.001 0.001 0.001
- link base_link: mass 4.00000000 -> None; geometry 
- link roll_front_left: geometry collision mesh filename=file:///home/andi/project/ros2_workspace/install/self_drivi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 scale=1 1 1; visual mesh filename=file:///home/andi/project/ros2_workspace/install/self_drivi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 scale=1 1 1
- link roll_front_right: geometry collision mesh filename=file:///home/andi/project/ros2_workspace/install/self_drivi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 scale=1 1 1; visual mesh filename=file:///home/andi/project/ros2_workspace/install/self_drivi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 scale=1 1 1
Joints:
- removed joint base_joint
- added joint base_footprint_joint: type fixed, parent base_link, child base_footprint, origin xyz=0 0 0.0 rpy=0 0 0
- added joint chassis_joint: type fixed, parent base_link, child chassis, origin xyz=0 0 0.5 rpy=0 0 0
- added joint control_joint: type fixed, parent chassis, child control, origin xyz=0 0 0.078 rpy=0 0 0
- joint camera_joint: parent base_link -> chassis
- joint lidar_joint: child lidar -> rplidar_link; parent base_link -> chassis
- joint roll_front_left_joint: parent base_link -> chassis
- joint roll_front_right_joint: parent base_link -> chassis
- joint wheel_back_left_joint: parent base_link -> chassis
- joint wheel_back_right_joint: parent base_link -> chassis

Commit message: driving_bot_simulation_navigation entfernt

File: urdf/ikea_table.urdf (robot description, URDF)
Before this commit: robot ikea_table, 12 links, 11 joints
Links:
- link control: geometry collision box size=0.075 0.30 0.075; visual box size=0.075 0.30 0.075
