Commit message: Box Robot Modell hinzugefügt

File: urdf/box_robot.urdf (robot description, URDF)
Before this commit: robot my_robot, 4 links, 3 joints
Links:
- added link lidar_mount, mass 0.05; collision box size=0.05 0.05 0.02; visual box size=0.05 0.05 0.02
- added link lidar_sensor, mass 0.02; collision cylinder length=0.01 radius=0.02; visual cylinder length=0.01 radius=0.02
- link front_ball: geometry collision sphere radius=0.015; visual sphere radius=0.015
Joints:
- added joint lidar_mount_joint: type fixed, parent base_link, child lidar_mount, origin xyz=0 0 0.04 rpy=0 0 0
- added joint lidar_sensor_joint: type fixed, parent lidar_mount, child lidar_sensor, origin xyz=0 0 0.14 rpy=0 0 0
- joint front_ball_joint: origin xyz=0.08 0 0.007 rpy=0 0 0 -> xyz=0.09 0 0.01 rpy=0 0 0

Commit message: es funktioniert erstmal

File: urdf/box_robot.urdf (robot description, URDF)
Before this commit: robot my_robot, 6 links, 5 joints
Links:
- removed link lidar_sensor
- added link base_footprint, mass 0.0001; visual box size=0.001 0.001 0.001
- added link base_laser, mass 0.02; collision cylinder length=0.01 radius=0.02; visual cylinder length=0.01 radius=0.02
Joints:
- removed joint lidar_sensor_joint
- added joint base_footprint_joint: type fixed, parent base_link, child base_footprint, origin xyz=0 0 0.0 rpy=0 0 0
- added joint base_laser_joint: type fixed, parent lidar_mount, child base_laser, origin xyz=0 0 0.14 rpy=0 0 0
